File: MCU Section.kicad_sch (KiCad schematic)
At the start: 75 parts, among them J4 Conn_01x04, U10 ESP32-C6-MINI-1-H8, U11 TLV62569ADRL, U12 XAL4020-222MEB, U13 GD25Q256EYIGR, U18 ESD5451N_C2936977, U8 ESD5451N_C2936977, U9 ESP32-P4NRW32_C22387510, X1 40MHz

Commit message: Finalize the schematic
Parts:
- removed C31, C34, C47, C58: 10uF, PCM_JLCPCB:C_0402, symbol PCM_JLCPCB-Capacitors:0402,10uF
- removed C40: 4.7uF, PCM_JLCPCB:C_0402, symbol PCM_JLCPCB-Capacitors:0402,4.7uF
- removed C61, C62: 18pF, PCM_JLCPCB:C_0402, symbol PCM_JLCPCB-Capacitors:0402,18pF
- added C31, C37: 18pF, Capacitor_SMD:C_0201_0603Metric, symbol Device:C_Small
- added C32, C33, C34, C35, C36: 10uF, Capacitor_SMD:C_0402_1005Metric, symbol Device:C_Small
- R13: renamed from R14; value 499k -> 100k
- R14: renamed from R13; value 499k -> 100k
Connections:
- net ESP_3V3: now also C33.1, C35.1, C36.1
- net ESP_VBAT: now also C32.1
- net ESP_VDD_HP: now also C34.1
- net GND: now also C31.1, C32.2, C33.2, C34.2, C35.2, C36.2, C37.1
- net XTAL_N: now also C31.2
- net XTAL_P: now also C37.2
Other:
- note added: "1.2 = 0.6*(1+R13/100)"
- note added: "Output Voltage"
- note added: "R13=100k"
- note added: "V_OUT = V_FB*(1+R13/R14)"
- moved on the sheet: C100, C101, C102, C103, C104, C105, C106, C107, C108, C109, C110, C111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

Commit message: Updated the net labels for 3v3 and sys rail
Connections:
- net VADC: now reaches U9.56 (GPIO27)
- net usb_vbus_det: now reaches U9.57 (GPIO28)
Changed lines of the file:
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@@
 	)
 	(junction
+		(at 157.48 196.85)
+		(diameter 0)
+		(color 0 0 0 0)
+	)
+	(junction
 		(at 166.37 250.19)
 		(diameter 0)
@@
 	)
 	(junction
-		(at 157.48 196.85)
-		(diameter 0)
-		(color 0 0 0 0)
-	)
-	(junction
 		(at 176.53 278.13)
 		(diameter 0)
@@
 		)
 	)
-	(polyline
-		(pts
-			(xy 247.396 190.754) (xy 247.396 195.326)
-		)
-		(stroke
-			(width 0)
-			(type default)
-		)
-	)
 	(wire
 		(pts
@@
 		)
 	)
-	(polyline
-		(pts
-			(xy 247.142 210.82) (xy 247.142 223.012)
-		)
-		(stroke
-			(width 0)
-			(type default)
-		)
-	)
 	(wire
 		(pts
@@
 		)
 	)
-	(polyline
-		(pts
-			(xy 246.888 284.226) (xy 246.888 290.068)
-		)
-		(stroke
-			(width 0)
-			(type default)
-		)
-	)
 	(wire
 		(pts
@@
 	(wire
 		(pts
+			(xy 251.46 298.45) (xy 245.11 298.45)
+		)
+		(stroke
+			(width 0)
+			(type default)
+		)
+	)
+	(wire
+		(pts
 			(xy 496.57 127) (xy 499.11 127)
 		)
@@
 		)
 	)
-	(polyline
-		(pts
-			(xy 247.142 198.882) (xy 247.142 207.772)
-		)
-		(stroke
-			(width 0)
-			(type default)
-		)
-	)
 	(wire
 		(pts
@@
 	(wire
 		(pts
+			(xy 251.46 295.91) (xy 245.11 295.91)
+		)
+		(stroke
+			(width 0)
+			(type default)
+		)
+	)
+	(wire
+		(pts
 			(xy 314.96 266.7) (xy 314.96 269.24)
 		)
@@
 		)
 	)
-	(polyline
-		(pts
-			(xy 247.142 226.314) (xy 247.142 238.252)
-		)
-		(stroke
-			(width 0)
-			(type default)
-		)
-	)
 	(wire
 		(pts
@@
 		)
 	)
+	(hierarchical_label "usb_vbus_det"
+		(shape input)
+		(at 251.46 295.91 0)
+		(effects
+			(font
+				(size 1.27 1.27)
+			)
+			(justify left)
+		)
+	)
 	(hierarchical_label "I2C1_SDA"
 		(shape input)
@@
 		)
 	)
+	(hierarchical_label "VADC"
+		(shape passive)
+		(at 251.46 298.45 0)
+		(effects
+			(font
+				(size 1.27 1.27)
+			)
+			(justify left)
+		)
+	)
 	(hierarchical_label "DSI_CLKN"
 		(shape output)
@@
 	)
 	(symbol
+		(lib_id "power:+3V3")
+		(at 157.48 196.85 0)
+		(unit 1)
+		(body_style 1)
+		(exclude_from_sim no)
+		(in_bom yes)
+		(on_board yes)
+		(in_pos_files yes)
+		(dnp no)
+		(property "Reference" "#PWR0235"
+			(at 157.48 200.66 0)
+			(hide yes)
+			(show_name no)
+			(do_not_autoplace no)
+			(effects
+				(font
+					(size 1.27 1.27)
+				)
+			)
+		)
+		(property "Value" "ESP_3V3"
+			(at 157.48 193.04 0)
+			(show_name no)
+			(do_not_autoplace no)
+			(effects
+				(font
+					(size 1.27 1.27)
+				)
+			)
+		)
+		(property "Footprint" ""
+			(at 157.48 196.85 0)
+			(hide yes)
+			(show_name no)
+			(do_not_autoplace no)
+			(effects
+				(font
+					(size 1.27 1.27)
+				)
+			)
+		)
+		(property "Datasheet" ""
+			(at 157.48 196.85 0)
+			(hide yes)
+			(show_name no)
+			(do_not_autoplace no)
+			(effects
+				(font
+					(size 1.27 1.27)
+				)
+			)
+		)
+		(property "Description" "Power symbol creates a global label with name \"+3V3\""
+			(at 157.48 196.85 0)
+			(hide yes)
+			(show_name no)
+			(do_not_autoplace no)
+			(effects
+				(font
+					(size 1.27 1.27)
+				)
+			)
+		)
+		(pin "1"
+		)
+		(instances
+			(project "Galatea Keyboard PCB"
+				(path "/04167948-25c2-4ca8-b9d8-855756010414/428647ab-2359-4bbe-93ac-b947dd4182f9"
+					(reference "#PWR0235")
+					(unit 1)
+				)
+			)
+		)
+	)
+	(symbol
 		(lib_id "power:GND")
 		(at 281.94 247.65 0)
@@
 					(unit 1)
 				)
-			)
-		)
-	)
-	(symbol
-		(lib_id "power:+3V3")
-		(at 157.48 196.85 0)
-		(unit 1)
-		(body_style 1)
-		(exclude_from_sim no)
-		(in_bom yes)
-		(on_board yes)
-		(in_pos_files yes)
-		(dnp no)
-		(property "Reference" "#PWR096"
-			(at 157.48 200.66 0)
-			(hide yes)
-			(show_name no)
-			(do_not_autoplace no)
-			(effects
-				(font
-					(size 1.27 1.27)
-				)
-			)
-		)
-		(property "Value" "ESP_3V3"
-			(at 157.48 193.04 0)
-			(show_name no)
-			(do_not_autoplace no)
-			(effects
-				(font
-					(size 1.27 1.27)
-				)
-			)
-		)
-		(property "Footprint" ""
-			(at 157.48 196.85 0)
-			(hide yes)
-			(show_name no)
-			(do_not_autoplace no)
-			(effects
-				(font
-					(size 1.27 1.27)
-				)
-			)
-		)
-		(property "Datasheet" ""
-			(at 157.48 196.85 0)
-			(hide yes)
-			(show_name no)
-			(do_not_autoplace no)
-			(effects
-				(font
-					(size 1.27 1.27)
-				)
-			)
-		)
-		(property "Description" "Power symbol creates a global label with name \"+3V3\""
-			(at 157.48 196.85 0)
-			(hide yes)
-			(show_name no)
-			(do_not_autoplace no)
-			(effects
-				(font
-					(size 1.27 1.27)
-				)
-			)
-		)
-		(pin "1"
-		)
-		(instances
-			(project "Galatea Keyboard PCB"
-				(path "/04167948-25c2-4ca8-b9d8-855756010414/428647ab-2359-4bbe-93ac-b947dd4182f9"
-					(reference "#PWR096")
-					(unit 1)
-				)

Commit message: Establish a comm protocol between C6 and P4. Also added programming headers
Parts:
- removed J4: Conn_01x04, Connector_PinHeader_2.54mm:PinHeader_1x04_P2.54mm_Vertical, symbol Connector_Generic:Conn_01x04
- added C117: 100nF, Capacitor_SMD:C_0201_0603Metric, symbol Device:C_Small
- added J2: Conn_02x03_Odd_Even, Connector_PinHeader_2.54mm:PinHeader_2x03_P2.54mm_Vertical, symbol Connector_Generic:Conn_02x03_Odd_Even
- added J3: Conn_01x04, Connector_PinHeader_2.54mm:PinHeader_1x04_P2.54mm_Vertical, symbol Connector_Generic:Conn_01x04
- added R50, R51: 0Ω, PCM_JLCPCB:R_0402, symbol PCM_JLCPCB-Resistors:0402,0Ω
- added R52: 10kΩ, PCM_JLCPCB:R_0603, symbol PCM_JLCPCB-Resistors:0603,10kΩ
Connections:
- net ESP_VBAT is gone; now on net ESP_3V3: C116.1, C32.1, U9.102 (VBAT)
- net C6_U0RXD: now also J2.4 (Pin_4)
- net C6_U0TXD: now also J2.3 (Pin_3)
- net ESP_3V3: now also J2.1 (Pin_1), J3.4 (Pin_4), R52.2
- net ESP_VDD_HP: now also U9.54 (NC), C117.1
- net GND: now also C117.2, J2.2 (Pin_2), J3.1 (Pin_1)
- net SDB: no longer U9.6 (GPIO6)
- net UART_RX: no longer U9.22 (GPIO20)
- net UART_TX: no longer U9.20 (GPIO19)
- net VADC: now also U9.93 (GPIO50); no longer U9.56 (GPIO27)
- net UART0_TXD: now reaches U9.69 (GPIO37)
- net UART0_TXD: now also J3.3 (Pin_3)
- net UART0_RXD: now reaches U9.70 (GPIO38)
- net UART0_RXD: now also J3.2 (Pin_2)
- net GPIO54: now reaches U9.98 (GPIO54)
- net GPIO54: now also R51.1
- net C6_IO12: now reaches U10.17 (IO12)
- net C6_IO13: now reaches U10.18 (IO13)
- net at U10.22 (IO8): now also R52.1
- net C6_IO9: now reaches U10.23 (IO9)
- net C6_IO9: now also J2.5 (Pin_5)
- net C6_IO2: now reaches U10.5 (IO2)
- net C6_IO2: now also R50.2
- net CHIP_PU renamed C6_CHIP_PU
- net C6_CHIP_PU: now also J2.6 (Pin_6), R51.2; no longer U9.23 (GPIO21)
- new net GPIO6: R50.1, U9.6 (GPIO6)
- no-connect marks 17 -> 24
Other:
- note added: "programming header"
- note removed: "STRAPPING PINS"
- note removed: "UART PROTOCOL"
- moved on the sheet: C100, C101, C102, C103, C104, C105, C106, C107, C108, C109, C110, C111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

Commit message: Did the layout plan
Parts:
- removed C14, C15: 100nF, Capacitor_SMD:C_0603_1608Metric, symbol Device:C_Small
- removed R42, R52: 10kΩ, PCM_JLCPCB:R_0603, symbol PCM_JLCPCB-Resistors:0603,10kΩ
- added C15, C38: 100nF, PCM_JLCPCB:C_0402, symbol PCM_JLCPCB-Capacitors:0402,100nF
- added R52, R53: 10kΩ, PCM_JLCPCB:R_0402, symbol PCM_JLCPCB-Resistors:0402,10kΩ
- J3: now not fitted; now left out of the parts list
Connections:
- net C6_CHIP_PU: now also R53.1
- net ESP_3V3: now also R52.2, R53.2
- net ESP_EN: now also C15.1
- net GND: now also C15.2, C38.2
- net GPIO_35: now also C38.1
- net at U10.22 (IO8): now also R52.1

Commit message: Progress on the PCB routing
Connections:
- net UART_RX is gone; now on net C6_U0RXD: U10.31 (TXD0)
- net UART_TX is gone; now on net C6_U0TXD: U10.30 (RXD0)
- net DSI_CLKN renamed DSI_CLK_N
- net DSI_CLKP renamed DSI_CLK_P
- net DSI_DATAN0 renamed DSI_DATA0_N
- net DSI_DATAN1 renamed DSI_DATA1_N
- net DSI_DATAP0 renamed DSI_DATA0_P
- net DSI_DATAP1 renamed DSI_DATA1_P
Changed lines of the file:
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@@
-		)
-	)
-	(label "UART_TX"
-		(at 453.39 81.28 0)
-		(effects
-			(font
-				(size 1.27 1.27)
-			)
-			(justify left bottom)
 		)
 	)
@@
 		)
 	)
+	(label "C6_U0TXD"
+		(at 453.39 81.28 0)
+		(effects
+			(font
+				(size 1.27 1.27)
+			)
+			(justify left bottom)
+		)
+	)
 	(label "ESP_EN"
 		(at 92.71 289.56 0)
@@
 		)
 	)
+	(label "C6_U0RXD"
+		(at 453.39 83.82 0)
+		(effects
+			(font
+				(size 1.27 1.27)
+			)
+			(justify left bottom)
+		)
+	)
 	(label "DSI_REXT"
 		(at 210.82 364.49 0)
@@
 		)
 	)
-	(label "UART_RX"
-		(at 453.39 83.82 0)
-		(effects
-			(font
-				(size 1.27 1.27)
-			)
-			(justify left bottom)
-		)
-	)
 	(label "DSI_REXT"
 		(at 180.34 303.53 0)
@@
 		)
 	)
-	(hierarchical_label "DSI_DATAN1"
+	(hierarchical_label "DSI_DATA1_N"
 		(shape output)
 		(at 189.23 308.61 180)
@@
 		)
 	)
-	(hierarchical_label "DSI_DATAP1"
+	(hierarchical_label "DSI_DATA1_P"
 		(shape output)
 		(at 189.23 306.07 180)
@@
 		)
 	)
-	(hierarchical_label "DSI_DATAN0"
+	(hierarchical_label "DSI_DATA0_N"
 		(shape output)
 		(at 189.23 316.23 180)
@@
 		)
 	)
-	(hierarchical_label "DSI_CLKP"
+	(hierarchical_label "DSI_CLK_P"
 		(shape output)
 		(at 189.23 313.69 180)
@@
 		)
 	)
-	(hierarchical_label "DSI_DATAP0"
+	(hierarchical_label "DSI_DATA0_P"
 		(shape output)
 		(at 189.23 318.77 180)
@@
 		)
 	)
-	(hierarchical_label "DSI_CLKN"
+	(hierarchical_label "DSI_CLK_N"
 		(shape output)
 		(at 189.23 311.15 180)

Commit message: Finalizing the routing
Connections:
- net +3V3 is gone; now on net ESP_3V3: R4.1
Changed lines of the file:
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@@
 	)
 	(symbol
-		(lib_id "power:+3V3")
-		(at 105.41 280.67 0)
-		(unit 1)
-		(body_style 1)
-		(exclude_from_sim no)
-		(in_bom yes)
-		(on_board yes)
-		(in_pos_files yes)
-		(dnp no)
-		(property "Reference" "#PWR040"
-			(at 105.41 284.48 0)
-			(hide yes)
-			(show_name no)
-			(do_not_autoplace no)
-			(effects
-				(font
-					(size 1.27 1.27)
-				)
-			)
-		)
-		(property "Value" "+3V3"
-			(at 105.41 277.368 0)
-			(show_name no)
-			(do_not_autoplace no)
-			(effects
-				(font
-					(size 1.27 1.27)
-				)
-			)
-		)
-		(property "Footprint" ""
-			(at 105.41 280.67 0)
-			(hide yes)
-			(show_name no)
-			(do_not_autoplace no)
-			(effects
-				(font
-					(size 1.27 1.27)
-				)
-			)
-		)
-		(property "Datasheet" ""
-			(at 105.41 280.67 0)
-			(hide yes)
-			(show_name no)
-			(do_not_autoplace no)
-			(effects
-				(font
-					(size 1.27 1.27)
-				)
-			)
-		)
-		(property "Description" "Power symbol creates a global label with name \"+3V3\""
-			(at 105.41 280.67 0)
-			(hide yes)
-			(show_name no)
-			(do_not_autoplace no)
-			(effects
-				(font
-					(size 1.27 1.27)
-				)
-			)
-		)
-		(pin "1"
-		)
-		(instances
-			(project "Galatea Keyboard PCB"
-				(path "/04167948-25c2-4ca8-b9d8-855756010414/428647ab-2359-4bbe-93ac-b947dd4182f9"
-					(reference "#PWR040")
-					(unit 1)
-				)
-			)
-		)
-	)
-	(symbol
 		(lib_id "power:GND")
 		(at 162.56 355.6 0)
@@
 					(unit 1)
 				)
+			)
+		)
+	)
+	(symbol
+		(lib_id "power:+3V3")
+		(at 105.41 280.67 0)
+		(unit 1)
+		(body_style 1)
+		(exclude_from_sim no)
+		(in_bom yes)
+		(on_board yes)
+		(in_pos_files yes)
+		(dnp no)
+		(property "Reference" "#PWR0263"
+			(at 105.41 284.48 0)
+			(hide yes)
+			(show_name no)
+			(do_not_autoplace no)
+			(effects
+				(font
+					(size 1.27 1.27)
+				)
+			)
+		)
+		(property "Value" "ESP_3V3"
+			(at 105.41 276.86 0)
+			(show_name no)
+			(do_not_autoplace no)
+			(effects
+				(font
+					(size 1.27 1.27)
+				)
+			)
+		)
+		(property "Footprint" ""
+			(at 105.41 280.67 0)
+			(hide yes)
+			(show_name no)
+			(do_not_autoplace no)
+			(effects
+				(font
+					(size 1.27 1.27)
+				)
+			)
+		)
+		(property "Datasheet" ""
+			(at 105.41 280.67 0)
+			(hide yes)
+			(show_name no)
+			(do_not_autoplace no)
+			(effects
+				(font
+					(size 1.27 1.27)
+				)
+			)
+		)
+		(property "Description" "Power symbol creates a global label with name \"+3V3\""
+			(at 105.41 280.67 0)
+			(hide yes)
+			(show_name no)
+			(do_not_autoplace no)
+			(effects
+				(font
+					(size 1.27 1.27)
+				)
+			)
+		)
+		(pin "1"
+		)
+		(instances
+			(project "Galatea Keyboard PCB"
+				(path "/04167948-25c2-4ca8-b9d8-855756010414/428647ab-2359-4bbe-93ac-b947dd4182f9"
+					(reference "#PWR0263")
+					(unit 1)
+				)

Commit message: Progressing with layout optimization
Parts:
- removed C101, C102, C103, C105, C106, C107, C108, C109, C110, C111, C112, C113, C114, C115, C116, C117: 100nF, Capacitor_SMD:C_0201_0603Metric, symbol Device:C_Small
- removed C104: 1uF, Capacitor_SMD:C_0201_0603Metric, symbol Device:C_Small
- removed C15, C38, C43: 100nF, PCM_JLCPCB:C_0402, symbol PCM_JLCPCB-Capacitors:0402,100nF
- removed C29: 10uF, PCM_JLCPCB:C_0805, symbol PCM_JLCPCB-Capacitors:0805,10uF
- removed C30: 100nF, PCM_JLCPCB:C_0603, symbol PCM_JLCPCB-Capacitors:0603,100nF
- removed C31, C37: 18pF, Capacitor_SMD:C_0201_0603Metric, symbol Device:C_Small
- removed C32, C33: 10uF, Capacitor_SMD:C_0402_1005Metric, symbol Device:C_Small
- removed X1: 40MHz, CN4040M00012T8188017:CRYSTAL-SMD_4P-L2.0-W1.6-BL, symbol CN4040M00012T8188017:CN4040M00012T8188017
- added C39, C48: 10nF, Capacitor_SMD:C_0402_1005Metric, symbol Device:C_Small
- added C40, C45, C46, C49, C50, C51, C52, C54, C55, C56, C57, C59, C60, C61, C62, C86, C87, C88, C89, C90: 100nF, Capacitor_SMD:C_0402_1005Metric, symbol Device:C_Small
- added C44, C53, C58: 10uF, Capacitor_SMD:C_0402_1005Metric, symbol Device:C_Small
- added C47, C91: 1uF, Capacitor_SMD:C_0402_1005Metric, symbol Device:C_Small
- added X1: XXDBBCNANF-40.000000MHZ, XXDBBCNANF-40.000000MHZ:CRYSTAL-SMD_4P-L3.2-W2.5-BL, symbol XXDBBCNANF-40.000000MHZ:XXDBBCNANF-40.000000MHZ
- C100, C99: value 100nF -> 10uF; footprint Capacitor_SMD:C_0201_0603Metric -> Capacitor_SMD:C_0402_1005Metric; LCSC C49062 -> (none); Package size 0201 -> (none); Voltage Rated 10V -> (none)
- C34: value 10uF -> 1uF
- C92: value 10nF -> 100nF; footprint Capacitor_SMD:C_0201_0603Metric -> Capacitor_SMD:C_0402_1005Metric; LCSC C76938 -> (none); Package size 0201 -> (none); Voltage Rated 25V -> (none)
- C93: value 100nF -> 18pF; footprint Capacitor_SMD:C_0201_0603Metric -> Capacitor_SMD:C_0402_1005Metric; LCSC C49062 -> (none); Package size 0201 -> (none); Voltage Rated 10V -> (none)
- C94: value 10nF -> 18pF; footprint Capacitor_SMD:C_0201_0603Metric -> Capacitor_SMD:C_0402_1005Metric; LCSC C76938 -> (none); Package size 0201 -> (none); Voltage Rated 25V -> (none)
- C95, C97: footprint Capacitor_SMD:C_0201_0603Metric -> Capacitor_SMD:C_0402_1005Metric; LCSC C49062 -> (none); Package size 0201 -> (none); Voltage Rated 10V -> (none)
- C96, C98: value 1uF -> 100nF; footprint Capacitor_SMD:C_0201_0603Metric -> Capacitor_SMD:C_0402_1005Metric; LCSC C76935 -> (none); Package size 0201 -> (none); Voltage Rated 10V -> (none)
Connections:
- net ESP_3V3: now also C98.1, C99.1, C48.1, C49.1, C50.1, C51.1, C52.1, C53.1, C54.1, C55.1, C58.1, C60.1, C61.1, C89.1; no longer C100.1, C92.1, C93.1, U9.85 (VDDPST_5)
- net ESP_EN: now also C96.1
- net ESP_VDD_HP: now also C92.1, C40.1, C44.1, C56.1, C59.1; no longer C34.1, C99.1
- net GND: now also C93.1, C94.1, C39.2, C40.2, C44.2, C45.2, C46.2, C47.2, C48.2, C49.2, C50.2, C51.2, C52.2, C53.2, C54.2, C55.2, C56.2, C57.2, C58.2, C59.2, C60.2, C61.2, C62.2, C86.2, C87.2, C88.2, C89.2, C90.2, C91.2, X1.2 (GND), X1.4 (GND); no longer C93.2, C94.2
- net GPIO_35: now also C97.1
- net VDDO_3: now also C39.1, C46.1, C47.1, C87.1; no longer C94.1, C95.1, C96.1
- net VDDO_4: now also C100.1, U9.85 (VDDPST_5), C57.1, C88.1
- net VDDO_FLASH: now also C62.1
- net VDDO_PSRAM: now also C86.1, C90.1, C91.1
- net VDD_FLASH: now also C34.1, C95.1, C45.1; no longer C97.1, C98.1
- net XTAL_N: now also C93.2, X1.3
- net XTAL_P: now also C94.2, X1.1

Commit message: Done with the routing. Yet to correct the issue raised and review the whole design
Parts:
- C100, C35, C36, C44, C53, C58: LCSC (none) -> C6119763
- C34, C47, C91: JLCPCB Part # (none) -> C52923
- C40, C45, C46, C49, C50, C51, C52, C54, C55, C56, C57, C59, C60, C61, C62, C86, C87, C88, C89, C90, C92, C95, C96, C97: JLCPCB Part # (none) -> C307331
- C41: LCSC (none) -> C1779
- C42: LCSC (none) -> C440198
- C98: footprint Capacitor_SMD:C_0402_1005Metric -> Capacitor_SMD:C_0603_1608Metric; LCSC (none) -> C14663
- C99: footprint Capacitor_SMD:C_0402_1005Metric -> Capacitor_SMD:C_0805_2012Metric; LCSC (none) -> C440198
- R13, R14: LCSC (none) -> C25803
- R16, R17: LCSC (none) -> C43251
- U11: LCSC (none) -> C398367
