File: RGB LEDs.kicad_sch (KiCad schematic)
At the start: 92 parts, among them U3 IS31FL3733B-QFLS4-TR

Commit message: Finalizing the routing
Parts:
- removed DW31, DW60, DW74, DW84: WHITE, LED_SMD:LED_0603_1608Metric, symbol Device:LED
Connections:
- net +3V3 renamed ESP_3V3
- net CS16: no longer names the net of U3.33 (CS16)
- no-connect marks 7 -> 8
