File: Galatea Keyboard PCB.kicad_pcb (KiCad board)
At the start: 4 copper layers, 404 x 142.3 mm, 451 parts, among them CN1 S2B-PH-SM4-TB, J1 USB_C_Receptacle_USB2.0, J2 Conn_02x03_Odd_Even, J3 Conn_01x04, Q1 MMBT3904, Q2 SSM3J328R,LF, SW1 EC11E18244AU, U1 TCA8418RTWR, U10 ESP32-C6-MINI-1-H8, U11 TLV62569ADRL, U12 XAL4020-222MEB, U13 GD25Q256EYIGR, U14 RT9193-18GB, U15 TPS63031DSK, U16 LPS3015-152MRC, U17 MAX17048G+T10, U18 ESD5451N_C2936977, U2 TCA8418RTWR, U3 IS31FL3733B-QFLS4-TR, U4 AP3032KTR-G1, U5 MP2617AGL-Z, U6 USBLC6-2SC6, U7 IS31FL3733B-QFLS4-TR, U8 ESD5451N_C2936977, U9 ESP32-P4NRW32_C22387510, X1 XXDBBCNANF-40.000000MHZ

Commit message: Corrected the issues raised
Parts:
- added R55: 10kΩ, PCM_JLCPCB:R_0603, B.Cu at (430.8, 144.9)
- added R56: 0Ω, PCM_JLCPCB:R_0402, B.Cu at (436.6, 150.5)
- added R57: 0Ω, PCM_JLCPCB:R_0402, B.Cu at (436.7, 149.2)
Connections:
- C62 pad 1: VDD_FLASH -> ESP_LDO_VO1
- FPC2 pad 26: RESET -> /MCU SECTION/LCD_RESET
- U9 pad 39: /MCU SECTION/DSI_DATA0_N -> /MCU SECTION/DSI_DATA0_P
- U9 pad 40: /MCU SECTION/DSI_DATA0_P -> /MCU SECTION/DSI_DATA0_N
- U9 pad 56: unconnected-(U9-GPIO27-Pad56) -> /MCU SECTION/LCD_RESET
- U9 pad 71: VDD_FLASH -> ESP_LDO_VO1
Routing:
- net /MCU SECTION/LCD_RESET: track 0.00 -> 48.4 mm, vias 0 -> 2
- net ESP_LDO_VO1: track 0.00 -> 21.4 mm, vias 0 -> 4
- net VDD_FLASH: track 36.6 -> 17.1 mm, vias 6 -> 2
- net /MCU SECTION/DSI_DATA0_P: track 61.4 -> 50.0 mm
- net /MCU SECTION/DSI_DATA0_N: track 60.7 -> 50.0 mm
- net GND: track 159.1 -> 160.3 mm, vias 717 -> 716
- net ESP_3V3: track 127.1 -> 128.2 mm, vias 66 -> 67
- net VCC_1.8V: track 12.4 -> 12.9 mm
