File: Galatea Keyboard PCB.kicad_pcb (KiCad board)
At the start: 4 copper layers, 404 x 142.3 mm, 454 parts, among them CN1 S2B-PH-SM4-TB, J1 USB_C_Receptacle_USB2.0, J2 Conn_02x03_Odd_Even, J3 Conn_01x04, Q1 MMBT3904, Q2 SSM3J328R,LF, SW1 EC11E18244AU, U1 TCA8418RTWR, U10 ESP32-C6-MINI-1-H8, U11 TLV62569ADRL, U12 XAL4020-222MEB, U13 GD25Q256EYIGR, U14 RT9193-18GB, U15 TPS63031DSK, U16 LPS3015-152MRC, U17 MAX17048G+T10, U18 ESD5451N_C2936977, U2 TCA8418RTWR, U3 IS31FL3733B-QFLS4-TR, U4 AP3032KTR-G1, U5 MP2617AGL-Z, U6 USBLC6-2SC6, U7 IS31FL3733B-QFLS4-TR, U8 ESD5451N_C2936977, U9 ESP32-P4NRW32_C22387510, X1 XXDBBCNANF-40.000000MHZ

Commit message: Prepare the production files, Included the 3D rendering images
Parts:
- R48: value 20.6k -> 20k
