File: Galatea Keyboard PCB.kicad_pcb (KiCad board)
At the start: 4 copper layers, 404 x 142.3 mm, 454 parts, among them CN1 S2B-PH-SM4-TB, J1 USB_C_Receptacle_USB2.0, J2 Conn_02x03_Odd_Even, J3 Conn_01x04, Q1 MMBT3904, Q2 SSM3J328R,LF, SW1 EC11E18244AU, U1 TCA8418RTWR, U10 ESP32-C6-MINI-1-H8, U11 TLV62569ADRL, U12 XAL4020-222MEB, U13 GD25Q256EYIGR, U14 RT9193-18GB, U15 TPS63031DSK, U16 LPS3015-152MRC, U17 MAX17048G+T10, U18 ESD5451N_C2936977, U2 TCA8418RTWR, U3 IS31FL3733B-QFLS4-TR, U4 AP3032KTR-G1, U5 MP2617AGL-Z, U6 USBLC6-2SC6, U7 IS31FL3733B-QFLS4-TR, U8 ESD5451N_C2936977, U9 ESP32-P4NRW32_C22387510, X1 XXDBBCNANF-40.000000MHZ

Commit message: Added GT911 connector and fix the USB_C issue
Parts:
- added FPC1: FH12-8S-0.5SH, FH12-8S-0.5SH(55):FPC-SMD_8P-P0.50_FH12S-8S-0.5SH-55, F.Cu at (446.7, 117.3)
- J1: value USB_C_Receptacle_USB2.0 -> Connector, USB-TYPE-C-16P; footprint PCM_marbastlib-various:USB_C_Receptacle_HRO_TYPE-C-31-M-12 -> PCM_JLCPCB:TYPE-C-SMD_HX-TYPE-C-16PIN
- moved J1 1.45 mm to (434.1, 105.9)
Connections:
- U9 pad 20: unconnected-(U9-GPIO19-Pad20) -> /MCU SECTION/CTP_INT
- U9 pad 22: unconnected-(U9-GPIO20-Pad22) -> /MCU SECTION/CTP_RST
Routing:
- net /KEYBOARD MATRIX/I2C1_SDA: track 161.0 -> 223.2 mm, vias 5 -> 7
- net /KEYBOARD MATRIX/I2C1_SCL: track 164.5 -> 226.5 mm, vias 6 -> 8
- net /MCU SECTION/CTP_INT: track 0.00 -> 54.0 mm, vias 0 -> 2
- net /MCU SECTION/CTP_RST: track 0.00 -> 53.3 mm, vias 0 -> 2
- net GND: track 160.3 -> 162.9 mm, vias 716 -> 701
- net ESP_3V3: track 128.2 -> 130.3 mm, vias 67 -> 69
- net Net-(B1-IO2): track 12.8 -> 11.7 mm
- net SYS: vias 4 -> 6
