File: Keyboard Matrix.kicad_sch (KiCad schematic)
At the start: 171 parts, among them U1 TCA8418RTWR, U2 TCA8418RTWR

Commit message: Updated the net labels for 3v3 and sys rail
Connections:
- net +3V3 renamed ESP_3V3

Commit message: Done with the routing. Yet to correct the issue raised and review the whole design
Parts:
- S3, S4: now not fitted; now left out of the parts list

Commit message: Done with the correction, PCB is complete
Parts:
- added R42, R54: 10k, Resistor_SMD:R_0603_1608Metric, symbol Device:R_Small
- added RN2: 10K, Resistor_SMD:R_Array_Convex_4x0402, symbol Device:R_Pack04_Split
Connections:
- net ESP_3V3: now also R42.1, R54.1, RN2.1 (R1.1), RN2.2 (R2.1), RN2.3 (R3.1), RN2.4 (R4.1)
- net I2C1_SCL: now also R54.2
- net I2C1_SDA: now also R42.2
- net at U2.14 (COL5): now also RN2.7 (R2.2)
- no-connect marks 0 -> 3
Other:
- note added: "Pull-ups"
