File: Rotary,tacts and LCD.kicad_sch (KiCad schematic)
At the start: 54 parts, among them Q1 MMBT3904, SW1 EC11E18244AU, U14 RT9193-18GB, U4 AP3032KTR-G1, U7 IS31FL3733B-QFLS4-TR

Commit message: Fix the issue on the display connector
Connections:
- net LEDA: now also C63.1, C64.1, D31.1, R25.1; no longer R26.1, R27.1
- net LEDK: now also R26.1, R27.1; no longer C63.1, C64.1, D31.1, R25.1
