File: Power Section.kicad_sch (KiCad schematic)
At the start: 53 parts, among them CN1 S2B-PH-SM4-TB, J1 USB_C_Receptacle_USB2.0, Q2 SSM3J328R,LF, U15 TPS63031DSK, U16 LPS3015-152MRC, U17 MAX17048, U5 MP2617AGL-Z, U6 USBLC6-2SC6

Commit message: Finalize thE battery Charging IC circuit
Parts:
- removed D86: SS54F, PCM_JLCPCB:D_SMAF, symbol PCM_JLCPCB-Diodes:Schottky,SS54F
- added R38: 10k, Resistor_SMD:R_0603_1608Metric, symbol Device:R_Small
- added R48: 20.6k, Resistor_SMD:R_0603_1608Metric, symbol Device:R_Small
- added R49: 100k, Resistor_SMD:R_0603_1608Metric, symbol Device:R_Small
Connections:
- net GND: now also U5.6 (~{EN}), U5.8 (M1), R38.2
- net VBUS: now also R48.1
- net VCC: now also R49.1
- net at J1.A4 (VBUS), J1.A9 (VBUS), J1.B4 (VBUS)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: now also B1.2 (IO2), C79.1, L2.1
- net at U5.19 (VLIM): now also R38.1, R48.2
- net at U5.7 (M0): now also R49.2
Other:
- note added: "Charge Current"
- note added: "I_CHG = 1971.42mA"
- note added: "I_CRG = 1.15*(1800/1.05k)mA"
- note added: "I_CRG = 1.15*(1800/R_SET)mA"
- note added: "Input Voltage Limit"
- note added: "V_IN_LIM = 1.52*((20.6+10)/10)V"
- note added: "V_IN_LIM = V_VLIM*((R1+R2)/R2)V"
- note added: "~ 2A"
- note added: "~4.65V"
- note removed: "I_SET = 1.15*(1800/1.05k)mA"
- note removed: "I_SET = 1.15*(1800/R_SET)mA"
- note removed: "I_SET = 1971.42mA"
- moved on the sheet: C18, C74, L3, R3, R37

Commit message: Updated the net labels for 3v3 and sys rail
Connections:
- net +3V3 is gone; now on net ESP_3V3: R39.1, R40.1, R41.1, TP15.1

Commit message: Did the layout plan
Parts:
- removed TP15, TP4, TP5: TestPoint, TestPoint:TestPoint_Pad_D1.5mm, symbol Connector:TestPoint
- removed U17: MAX17048, Abhishek_Library:SON50P200X200X80-9N, symbol PCM_marbastlib-various:MAX17048
- added U17: MAX17048G+T10, MAX17048:TDFN-8_L2.0-W2.0-P0.50-BL-EP1.2, symbol MAX17048:MAX17048G+T10
Connections:
- net +BATT: now also U17.2 (CELL), U17.3 (VDD)
- net ALERT: now also U17.5 (~{ALRT})
- net GND: now also U17.1 (CTG), U17.4 (GND), U17.6 (QSTRT), U17.9 (EP)
- net I2C0_SCL: now also U17.7 (SCL)
- net I2C0_SDA: now also U17.8 (SDA)
Other:
- moved on the sheet: C76, C77, R39, R40, R41, TP11

Commit message: Done with the routing. Yet to correct the issue raised and review the whole design
Parts:
- C16, C75, C84: LCSC (none) -> C14663
- C18, C85: LCSC (none) -> C15849
- R35, R36, R38: LCSC (none) -> C49330116
- R39, R40, R41: LCSC C177644 -> C49330116
- R49: LCSC (none) -> C25803
- U15: LCSC Part (none) -> C15516

Commit message: Done with the correction, PCB is complete
Parts:
- removed L2: BLM18PG121SN1D, BLM18PG121SN1D:L0603, symbol BLM18PG121SN1D:BLM18PG121SN1D_C14709
- added C29: 22uF, PCM_JLCPCB:C_0805, symbol PCM_JLCPCB-Capacitors:0805,22uF
- added L2: BLM18SG121TN1D, BLM18SG121TN1D:L0603, symbol BLM18SG121TN1D:BLM18SG121TN1D
- C75: value 100nF -> 200nF; LCSC C14663 -> (none)
Connections:
- net GND: now also U15.7 (PS/SYNC), C29.2
- net SYS: now also C16.1, U15.6 (EN), U15.8 (VINA), C29.1
- net VBUS: now also L2.2
- net at B1.2 (IO2), C79.1, J1.A4 (VBUS)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: now also L2.1
Other:
- moved on the sheet: C16

Commit message: Prepare the production files, Included the 3D rendering images
Parts:
- C71, C72, C73: LCSC (none) -> C344022
- C74: LCSC (none) -> C89632
- C75: LCSC (none) -> C3833176
- D59: LCSC (none) -> C2290
- D60: LCSC (none) -> C2286
- R3, R37: LCSC (none) -> C4109
- R48: value 20.6k -> 20k; LCSC (none) -> C4184
- R7: LCSC (none) -> C177342
- R8: LCSC (none) -> C22832
- TP11: now not fitted; now left out of the parts list
Changed lines of the file:
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@@
 			)
 		)
-		(property "Value" "20.6k"
+		(property "Value" "20k"
 			(at 161.29 152.4 0)
 			(show_name no)
@@
 			)
 		)
+		(property "LCSC" "C4184"
+			(at 158.75 151.13 0)
+			(hide yes)
+			(show_name no)
+			(do_not_autoplace no)
+			(effects
+				(font
+					(size 1.27 1.27)
+				)
+			)
+		)
 		(pin "1"
 		)
@@
 			)
 		)
+		(property "LCSC" "C2290"
+			(at 100.33 194.31 0)
+			(hide yes)
+			(show_name no)
+			(do_not_autoplace no)
+			(effects
+				(font
+					(size 1.27 1.27)
+				)
+			)
+		)
 		(pin "1"
 		)
@@
 			)
 		)
+		(property "LCSC" "C89632"
+			(at 57.15 180.34 0)
+			(hide yes)
+			(show_name no)
+			(do_not_autoplace no)
+			(effects
+				(font
+					(size 1.27 1.27)
+				)
+			)
+		)
 		(pin "2"
 		)
@@
 			)
 		)
+		(property "LCSC" "C344022"
+			(at 344.17 74.93 0)
+			(hide yes)
+			(show_name no)
+			(do_not_autoplace no)
+			(effects
+				(font
+					(size 1.27 1.27)
+				)
+			)
+		)
 		(pin "2"
 		)
@@
 			)
 		)
+		(property "LCSC" "C4109"
+			(at 87.63 191.77 90)
+			(hide yes)
+			(show_name no)
+			(do_not_autoplace no)
+			(effects
+				(font
+					(size 1.27 1.27)
+				)
+			)
+		)
 		(pin "2"
 		)
@@
 			)
 		)
-		(property "LCSC" ""
+		(property "LCSC" "C3833176"
 			(at 143.51 176.53 90)
 			(hide yes)
@@
 			)
 		)
+		(property "LCSC" "C177342"
+			(at 149.86 179.07 90)
+			(hide yes)
+			(show_name no)
+			(do_not_autoplace no)
+			(effects
+				(font
+					(size 1.27 1.27)
+				)
+			)
+		)
 		(pin "2"
 		)
@@
 		(body_style 1)
 		(exclude_from_sim no)
-		(in_bom yes)
+		(in_bom no)
 		(on_board yes)
 		(in_pos_files yes)
-		(dnp no)
+		(dnp yes)
 		(property "Reference" "TP11"
 			(at 380.746 208.28 90)
@@
 			)
 		)
+		(property "LCSC" "C344022"
+			(at 334.01 74.93 0)
+			(hide yes)
+			(show_name no)
+			(do_not_autoplace no)
+			(effects
+				(font
+					(size 1.27 1.27)
+				)
+			)
+		)
 		(pin "2"
 		)
@@
 			)
 		)
+		(property "LCSC" "C4109"
+			(at 82.55 194.31 90)
+			(hide yes)
+			(show_name no)
+			(do_not_autoplace no)
+			(effects
+				(font
+					(size 1.27 1.27)
+				)
+			)
+		)
 		(pin "2"
 		)
@@
 			)
 		)
+		(property "LCSC" "C344022"
+			(at 276.86 74.93 0)
+			(hide yes)
+			(show_name no)
+			(do_not_autoplace no)
+			(effects
+				(font
+					(size 1.27 1.27)
+				)
+			)
+		)
 		(pin "2"
 		)
@@
 			)
 		)
+		(property "LCSC" "C2286"
+			(at 95.25 191.77 0)
+			(hide yes)
+			(show_name no)
+			(do_not_autoplace no)
+			(effects
+				(font
+					(size 1.27 1.27)
+				)
+			)
+		)
 		(pin "1"
 		)
@@
 			(at 144.78 184.15 90)
 			(hide yes)
+			(show_name no)
+			(do_not_autoplace no)
+			(effects
+				(font
+					(size 1.27 1.27)
+				)
+			)
+		)
+		(property "LCSC" "C22832"
+			(at 144.78 184.15 90)
+			(hide yes)

Commit message: Added GT911 connector and fix the USB_C issue
Parts:
- removed J1: USB_C_Receptacle_USB2.0, PCM_marbastlib-various:USB_C_Receptacle_HRO_TYPE-C-31-M-12, symbol Connector:USB_C_Receptacle_USB2.0
- added J1: Connector, USB-TYPE-C-16P, PCM_JLCPCB:TYPE-C-SMD_HX-TYPE-C-16PIN, symbol PCM_JLCPCB-Extended:Connector, USB-TYPE-C-16P
Connections:
- net GND: now also J1.A12B1 (GND), J1.B12A1 (GND), J1.S1 (SHIELD)
- net USB+: now also J1.A6 (D+), J1.B6 (D+)
- net USB-: now also J1.A7 (D-), J1.B7 (D-)
- net at B1.2 (IO2), C79.1, L2.1: now also J1.A9B4 (VBUS), J1.B9A4 (VBUS)
- net at R5.1: now also J1.A5 (CC1)
- net at R6.1: now also J1.B5 (CC2)

Commit message: Added the connector and generated updated production files
Parts:
- removed TP11: TestPoint, TestPoint:TestPoint_Pad_D1.5mm, symbol Connector:TestPoint
